File: hardware/board/DeadHorsePCB.brd (EAGLE design)
At the start: 75.4 x 78.5 mm, 23 parts, among them J1 DIN5, Q1 BSS138, Q2 BSS138

Commit message: Further board modifications
Parts:
- moved R13 67.1 mm to (67.6, 66.5), turned to 270 degrees
- moved R7 64.8 mm to (67.6, 74.2), turned to 90 degrees
- moved R5 64.5 mm to (67.6, 58.9), turned to 270 degrees
- moved R8 64.4 mm to (67.6, 51.3), turned to 90 degrees
- moved R2 58.3 mm to (62.0, 36.1), turned to 90 degrees
- moved R10 51.2 mm to (67.6, 43.7), turned to 270 degrees
- moved R4 51.2 mm to (62.0, 43.7), turned to 270 degrees
- moved R12 46.9 mm to (62.0, 66.5), turned to 90 degrees
- moved R3 44.0 mm to (62.0, 74.2), turned to 270 degrees
- moved R11 42.8 mm to (62.0, 28.4), turned to 270 degrees
- moved R9 37.0 mm to (67.6, 36.1), turned to 270 degrees
- moved R6 31.3 mm to (62.0, 58.9), turned to 90 degrees
- moved R1 31.0 mm to (62.0, 51.3), turned to 90 degrees
- moved SELECT_BUTTON 20.5 mm to (23.9, 23.1)
- moved Q2 19.2 mm to (26.7, 39.4)
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Other:
- board size 75.4 x 78.5 mm -> 75.4 x 63.2 mm
- board text added: "CS"
- board text added: "DC"
- board text added: "RES"
- board text added: "SCK"

Commit message: Getting closer on the PCB
Parts:
- removed S1: ENCODER-SWITCH, SparkFun-Switches:ROTARY_ENC_PLAIN
- added ENCODER: (no value), con-lstb:MA05-1
- PLAY_BUTTON: value PlayButton -> PlayBtn
- SELECT_BUTTON: value SelectButton -> SelectBtn
- moved R6 56.8 mm to (36.6, 8.13)
- moved R5 54.3 mm to (57.4, 5.59)
- moved R12 52.4 mm to (49.3, 15.7)
- moved SELECT_BUTTON 51.0 mm to (41.9, 70.9), turned to 270 degrees
- moved R3 48.4 mm to (46.7, 28.2), turned to 0 degrees
- moved R11 46.4 mm to (46.5, 72.1), turned to 0 degrees
- moved R1 46.0 mm to (67.1, 5.59)
- moved J1 45.7 mm to (86.9, 78.5), flipped to the top
- moved R10 37.5 mm to (46.5, 74.7), turned to 180 degrees
- moved OLED 37.4 mm to (41.9, 42.9), turned to 90 degrees
- moved R4 37.0 mm to (51.8, 8.13)
- moved PLAY_BUTTON 35.3 mm to (41.9, 58.9), turned to 270 degrees
- moved TRELLIS 34.0 mm to (41.9, 26.7), turned to 270 degrees
- moved R9 32.0 mm to (46.5, 60.2), turned to 0 degrees
- moved Q2 31.8 mm to (41.9, 11.4)
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Connections:
- removed net N$11: OLED.5, U$8.39/A20
- removed net N$15: S1.B, U$8.24
- removed net N$17: S1.A, U$8.25
- removed net N$19: R11.1, SELECT_BUTTON.2, U$8.8
- new net CS: OLED.7, U$8.8
- new net DC: OLED.6, U$8.9
- new net N$22: R11.1, SELECT_BUTTON.2, U$8.3
- new net RES: OLED.5, U$8.10
- net GND: now also ENCODER.1, ENCODER.2; no longer S1.C, S1.SW+
- net N$10: now also ENCODER.5, U$8.16/A2; no longer OLED.6, U$8.38/A19
- net N$13: now also U$8.4; no longer U$8.9
- net N$14: now also U$8.5; no longer U$8.10
- net N$16: now also U$8.2; no longer U$8.7
- net N$20: now also ENCODER.3, U$8.18/A4; no longer S1.SW-, U$8.26
- net N$6: now also U$8.14/A0; no longer U$8.18/A4
- net N$7: now also U$8.15/A1; no longer U$8.19/A5
- net N$9: now also ENCODER.4, U$8.17/A3; no longer OLED.7, U$8.37/A18
Other:
- board size 75.4 x 63.2 mm -> 83.1 x 63.2 mm

Commit message: Added Ground Plane
Parts:
- ENCODER: value (none) -> ENCODER
- moved R6 45.9 mm to (67.1, 42.4), flipped to the bottom, turned to 180 degrees
- moved R5 41.1 mm to (62.0, 46.5), flipped to the bottom, turned to 0 degrees
- moved R1 40.9 mm to (67.1, 46.5), flipped to the bottom, turned to 180 degrees
- moved R12 40.7 mm to (75.9, 46.5), flipped to the bottom, turned to 0 degrees
- moved Q1 37.6 mm to (63.5, 27.2), flipped to the bottom
- moved R4 35.8 mm to (62.0, 42.4), flipped to the bottom, turned to 0 degrees
- moved Q2 31.8 mm to (63.5, 34.8), flipped to the bottom
- moved ENCODER 2.54 mm to (80.5, 49.3)
- moved R2 2.54 mm to (46.7, 33.0), flipped to the bottom, turned to 0 degrees
- flipped R10 to the bottom, turned to 0 degrees
- flipped R11 to the bottom, turned to 180 degrees
- flipped R13 to the bottom, turned to 0 degrees
- flipped R3 to the bottom, turned to 180 degrees
- flipped R7 to the bottom, turned to 0 degrees
- flipped R8 to the bottom, turned to 0 degrees
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Routing:
- net 3.3V: track 0.00 -> 133.7 mm
- net VIN: track 0.00 -> 101.6 mm
- net N$4: track 0.00 -> 70.6 mm, vias 0 -> 1
- net N$5: track 0.00 -> 39.2 mm, vias 0 -> 2
- net N$3: track 0.00 -> 37.2 mm, vias 0 -> 1
- net SCK: track 0.00 -> 30.5 mm
- net N$2: track 0.00 -> 25.6 mm
- net N$8: track 0.00 -> 25.2 mm, vias 0 -> 2
- net N$22: track 0.00 -> 19.2 mm
- net N$14: track 0.00 -> 18.2 mm
- net N$20: track 0.00 -> 17.2 mm
- net SDA: track 0.00 -> 15.0 mm
- net RES: track 0.00 -> 15.0 mm
- net DC: track 0.00 -> 15.0 mm
- net CS: track 0.00 -> 15.0 mm
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- added copper zone on layer 16, net GND
Other:
- board size 83.1 x 63.2 mm -> 67.8 x 63.2 mm
- board text added: "A"
- board text added: "B"
